File: PCB Design/STM32/stm32.sch (EAGLE design)
At the start: 54 parts, among them T1 SFH303, T2 SFH303, T3 SFH303, T4 SFH303, U1 MPU-6000QFN-24, U2 STM32F103RET6

Commit message: board making
Parts:
- removed C22: 10nF, SparkFun-Capacitors:CAP0402-CAP
- removed OSC: 8MHz, SparkFun2:CRYSTAL5X3
- removed R11: (no value), resistor:R-US_R0603
- removed R12: 42 Ohm, resistor:R-US_R0603
- removed U$2: MCP1700T-3302E/TT, Microchip_By_element14_Batch_1:MCP1700T-3302E/TT
- added C3: 4.7uF, SparkFun-Capacitors:CAP0603-CAP
- added Q5: (no value), semicon-smd-ipc:NPN-TRANSISTIOR-2COLSOT89
- added R1, R2: 10k, SparkFun-Passives:RESISTOR0402-RES
- added U4: MPU-6000QFN-24, SparkFun-Sensors:MPU-6000QFN-24
- C1: value 33pF -> 10nF; device SparkFun:CAP0402 -> SparkFun-Capacitors:CAP0603-CAP
- C10: value 10nF -> 22uF; device SparkFun-Capacitors:CAP0402-CAP -> rcl:CPOL-EUUD-4X5,8
- C11: value 100nF -> 22uF; device SparkFun-Capacitors:CAP0402-CAP -> rcl:CPOL-EUUD-4X5,8
- C12, C13: value 100nF -> 33pF; device SparkFun-Capacitors:CAP0402-CAP -> SparkFun:CAP0603
- C14: value 2.2nF -> 10uF; device SparkFun-Capacitors:CAP0402-CAP -> SparkFun-Capacitors:CAP_POL1206
- C15: value 0.1uF -> 10uF; device SparkFun-Capacitors:CAP0402-CAP -> SparkFun-Capacitors:CAP_POL1206
- C16: device SparkFun-Capacitors:CAP0402-CAP -> SparkFun-Capacitors:CAP0603-CAP
- C17, C19: value 10uF -> 0.1uF; device SparkFun-Capacitors:CAP_POL1206 -> SparkFun-Capacitors:CAP0603-CAP
- C18: value 0.1uF -> 10uF; device SparkFun-Capacitors:CAP0402-CAP -> SparkFun-Capacitors:CAP0603-CAP
- C2: value 33pF -> 1uF; device SparkFun:CAP0402 -> SparkFun-Capacitors:CAP0603-CAP
- C20: value 100nF -> 2.2nF; device SparkFun-Capacitors:CAP0402-CAP -> SparkFun-Capacitors:CAP0603-CAP
- C21: value 4.7uF -> 10nF; device SparkFun-Capacitors:CAP0402-CAP -> SparkFun-Capacitors:CAP0603-CAP
- C4, C5, C7: value 22uF -> 100nF; device rcl:CPOL-EUUD-4X5,8 -> SparkFun-Capacitors:CAP0603-CAP
- C6: value 1uF -> 100nF; device SparkFun:CAP0402 -> SparkFun-Capacitors:CAP0603-CAP
- C8: device SparkFun-Capacitors:CAP0402-CAP -> SparkFun:CAP0603
- C9: value 10uF -> 22uF; device SparkFun-Capacitors:CAP0402-CAP -> rcl:CPOL-EUUD-4X5,8
- Q1: value (none) -> 8MHz; device semicon-smd-ipc:NPN-TRANSISTIOR-2COLSOT89 -> SparkFun2:CRYSTAL5X3
- R3, R4: value 10k -> (none); device SparkFun-Passives:RESISTOR0402-RES -> resistor:R-US_R0603
- R7: value (none) -> 42 Ohm
- U1: value MPU-6000QFN-24 -> STM32F103RET6; device SparkFun-Sensors:MPU-6000QFN-24 -> ST Microelctronics_By_element14_Batch_1:STM32F103RET6
- U2: value STM32F103RET6 -> MCP1700T-3302E/TT; device ST Microelctronics_By_element14_Batch_1:STM32F103RET6 -> Microchip_By_element14_Batch_1:MCP1700T-3302E/TT
- USART: device SparkFun-Connectors:M03LOCK -> SparkFun-Connectors:M04LOCK
- renumbered D2 to D1, M1 to JP3, M2 to JP4, U$1 to U5, U$3 to U3
Connections:
- removed net N$11: SWD.4
- removed net N$12: SWD.3
- removed net N$13: SWD.2
- removed net N$18: SWD.1
- removed net N$8: SWD.5
- net GND: now also C1.2, C10.-, C11.-, C12.1, C13.1, C14.-, C15.-, C17.2, C19.2, C2.2, C3.2, C4.2, C5.2, C6.2, C7.2, C8.1, C9.-, R7.1, SWD.1, U1.BOOT0, U1.PB1_2, U1.VSSA, U1.VSS_1, U1.VSS_2, U1.VSS_3, U1.VSS_4, U2.GND, U4.AD0/SDO, U4.CLKIN, U4.FSYNC, U4.GND; no longer C1.1, C10.2, C11.2, C12.2, C13.2, C14.2, C15.2, C17.-, C19.-, C2.1, C22.2, C4.-, C5.-, C6.1, C7.-, C8.2, C9.2, R12.1, U$2.GND, U1.AD0/SDO, U1.CLKIN, U1.FSYNC, U1.GND, U2.BOOT0, U2.PB1_2, U2.VSSA, U2.VSS_1, U2.VSS_2, U2.VSS_3, U2.VSS_4
- net I2C1_SCL: now also R1.1, U1.PB6, U4.SCL/SCLK; no longer R3.1, U1.SCL/SCLK, U2.PB6
- net I2C1_SDA: now also R2.1, U1.PB7, U4.SDA/SDI; no longer R4.1, U1.SDA/SDI, U2.PB7
- net I2C1_SMBA: now also U1.PB5; no longer U2.PB5
- net INT: now also U1.PB8, U4.INT; no longer U1.INT, U2.PB8
- net IR_IN1: now also R7.2, T1.E, U1.PC0; no longer R9.2, T4.E, U2.PC0
- net IR_IN2: now also T2.E, U1.PC1; no longer T1.E, U2.PC1
- net IR_IN3: now also R9.2, T3.E, U1.PC2; no longer R10.2, T2.E, U2.PC2
- net IR_IN4: now also R10.2, T4.E, U1.PC3; no longer R12.2, T3.E, U2.PC3
- net IR_OUT1: now also Q2.B, U1.PC6; no longer Q1.B, U2.PC6
- net IR_OUT2: now also Q3.B, U1.PC7; no longer Q2.B, U2.PC7
- net IR_OUT3: now also Q4.B, U1.PC8; no longer Q3.B, U2.PC8
- net IR_OUT4: now also Q5.B, U1.PC9; no longer Q4.B, U2.PC9
- net JTAG-TCK: now also SWD.3, U1.PA14; no longer U2.PA14
- net JTAG-TDI: now also U1.PA15; no longer U2.PA15
- net JTAG-TDO: now also SWD.2, U1.PB3; no longer U2.PB3
- net JTAG-TMS: now also SWD.4, U1.PA13; no longer U2.PA13
- net JTAG-TRST: now also U1.PB4; no longer U2.PB4
- net M1CA: now also U1.PB12; no longer U2.PB12
- net M1CB: now also U1.PB13; no longer U2.PB13
- net M1I1: now also U1.PA3; no longer U2.PA3
- net M1I2: now also U1.PA2; no longer U2.PA2
- net M1P: now also U1.PA1; no longer U2.PA1
- net M2CA: now also U1.PB14; no longer U2.PB14
- net M2CB: now also U1.PB15; no longer U2.PB15
- net M2I1: now also U1.PA4; no longer U2.PA4
- net M2I2: now also U1.PA5; no longer U2.PA5
- net M2P: now also U1.PA6; no longer U2.PA6
- net N$1: now also C8.2, C9.+, U2.VIN; no longer C6.2, C7.+, U$2.VIN
- net N$10: now also C18.1, U4.REGOUT; no longer C9.1, U1.REGOUT
- net N$14: now also Q2.E; no longer Q1.E
- net N$15: now also Q3.E; no longer Q2.E
- net N$16: now also Q4.E; no longer Q3.E
- net N$17: now also Q5.E; no longer Q4.E
- net N$2: now also C13.2, Q1.1, U1.PD1_OSC_OUT; no longer C2.2, OSC.1, U2.PD1_OSC_OUT
- net N$3: now also Q2.C/, R3.1; no longer Q1.C/, R5.1
- net N$4: now also Q3.C/, R4.1; no longer Q2.C/, R6.1
- net N$5: now also Q4.C/, R5.1; no longer Q3.C/, R7.1
- net N$6: now also C12.2, Q1.2, U1.PD0_OSC_IN; no longer C1.2, OSC.2, U2.PD0_OSC_IN
- net N$7: now also Q5.C, R6.1; no longer Q4.C, R11.1
- net N$9: now also C20.1, U4.CPOUT; no longer C14.1, U1.CPOUT
- net RST: now also SWD.5, U1.NRST; no longer U2.NRST
- net USART1_CK: now also U1.PA8; no longer U2.PA8
- net USART1_CTS: now also U1.PA11; no longer U2.PA11
- net USART1_RTS: now also U1.PA12; no longer U2.PA12
- net USART1_RX: now also U1.PA10; no longer U2.PA10
- net USART1_TX: now also U1.PA9; no longer U2.PA9
- net VCC: now also C11.+, C14.+, C17.1, C3.1, C4.1, C5.1, C6.1, C7.1, R1.2, R2.2, U1.VDD_1, U1.VDD_2, U1.VDD_3, U1.VDD_4, U4.CS, U4.VDD, USART.4; no longer C10.1, C11.1, C12.1, C13.1, C15.1, C17.+, C20.1, C4.+, R11.2, R7.2, U1.CS, U1.VDD, U2.VDD_1, U2.VDD_2, U2.VDD_3, U2.VDD_4
- net VDD: now also C1.1, C10.+, C2.1, U1.VDDA, U2.VOUT; no longer C22.1, C5.+, C8.1, U$2.VOUT, U2.VDDA
- net V_BATT: now also C15.+, C19.1; no longer C18.1, C19.+
Other:
- moved on the sheet: C1, C12, C13, C16, C18, C2, C20, C21, C6, C8, Q2, Q3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

Commit message: board update
Connections:
- net I2C1_SCL renamed N$11
Changed lines of the file:
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@@
 <grid distance="0.1" unitdist="inch" unit="inch" style="lines" multiple="1" display="no" altdistance="0.01" altunitdist="inch" altunit="inch"/>
 <layers>
-<layer number="1" name="Top" color="4" fill="1" visible="yes" active="no"/>
-<layer number="2" name="Route2" color="1" fill="3" visible="yes" active="no"/>
-<layer number="3" name="Route3" color="4" fill="3" visible="yes" active="no"/>
-<layer number="14" name="Route14" color="1" fill="6" visible="yes" active="no"/>
-<layer number="15" name="Route15" color="4" fill="6" visible="yes" active="no"/>
-<layer number="16" name="Bottom" color="1" fill="1" visible="yes" active="no"/>
-<layer number="17" name="Pads" color="2" fill="1" visible="yes" active="no"/>
-<layer number="18" name="Vias" color="2" fill="1" visible="yes" active="no"/>
-<layer number="19" name="Unrouted" color="6" fill="1" visible="yes" active="no"/>
-<layer number="20" name="Dimension" color="15" fill="1" visible="yes" active="no"/>
-<layer number="21" name="tPlace" color="7" fill="1" visible="yes" active="no"/>
-<layer number="22" name="bPlace" color="7" fill="1" visible="yes" active="no"/>
-<layer number="23" name="tOrigins" color="15" fill="1" visible="yes" active="no"/>
-<layer number="24" name="bOrigins" color="15" fill="1" visible="yes" active="no"/>
-<layer number="25" name="tNames" color="7" fill="1" visible="yes" active="no"/>
-<layer number="26" name="bNames" color="7" fill="1" visible="yes" active="no"/>
-<layer number="27" name="tValues" color="7" fill="1" visible="yes" active="no"/>
-<layer number="28" name="bValues" color="7" fill="1" visible="yes" active="no"/>
+<layer number="1" name="Top" color="4" fill="1" visible="no" active="no"/>
+<layer number="2" name="Route2" color="1" fill="3" visible="no" active="no"/>
+<layer number="3" name="Route3" color="4" fill="3" visible="no" active="no"/>
+<layer number="14" name="Route14" color="1" fill="6" visible="no" active="no"/>
+<layer number="15" name="Route15" color="4" fill="6" visible="no" active="no"/>
+<layer number="16" name="Bottom" color="1" fill="1" visible="no" active="no"/>
+<layer number="17" name="Pads" color="2" fill="1" visible="no" active="no"/>
+<layer number="18" name="Vias" color="2" fill="1" visible="no" active="no"/>
+<layer number="19" name="Unrouted" color="6" fill="1" visible="no" active="no"/>
+<layer number="20" name="Dimension" color="15" fill="1" visible="no" active="no"/>
+<layer number="21" name="tPlace" color="7" fill="1" visible="no" active="no"/>
+<layer number="22" name="bPlace" color="7" fill="1" visible="no" active="no"/>
+<layer number="23" name="tOrigins" color="15" fill="1" visible="no" active="no"/>
+<layer number="24" name="bOrigins" color="15" fill="1" visible="no" active="no"/>
+<layer number="25" name="tNames" color="7" fill="1" visible="no" active="no"/>
+<layer number="26" name="bNames" color="7" fill="1" visible="no" active="no"/>
+<layer number="27" name="tValues" color="7" fill="1" visible="no" active="no"/>
+<layer number="28" name="bValues" color="7" fill="1" visible="no" active="no"/>
 <layer number="29" name="tStop" color="7" fill="3" visible="no" active="no"/>
 <layer number="30" name="bStop" color="7" fill="6" visible="no" active="no"/>
@@
 <layer number="35" name="tGlue" color="7" fill="4" visible="no" active="no"/>
 <layer number="36" name="bGlue" color="7" fill="5" visible="no" active="no"/>
-<layer number="37" name="tTest" color="7" fill="1" visible="yes" active="no"/>
-<layer number="38" name="bTest" color="7" fill="1" visible="yes" active="no"/>
+<layer number="37" name="tTest" color="7" fill="1" visible="no" active="no"/>
+<layer number="38" name="bTest" color="7" fill="1" visible="no" active="no"/>
 <layer number="39" name="tKeepout" color="4" fill="11" visible="no" active="no"/>
 <layer number="40" name="bKeepout" color="1" fill="11" visible="no" active="no"/>
@@
 <layer number="44" name="Drills" color="7" fill="1" visible="no" active="no"/>
 <layer number="45" name="Holes" color="7" fill="1" visible="no" active="no"/>
-<layer number="46" name="Milling" color="3" fill="1" visible="yes" active="no"/>
-<layer number="47" name="Measures" color="7" fill="1" visible="yes" active="no"/>
-<layer number="48" name="Document" color="7" fill="1" visible="yes" active="no"/>
-<layer number="49" name="Reference" color="7" fill="1" visible="yes" active="no"/>
-<layer number="50" name="dxf" color="7" fill="1" visible="yes" active="no"/>
-<layer number="51" name="tDocu" color="7" fill="1" visible="yes" active="no"/>
-<layer number="52" name="bDocu" color="7" fill="1" visible="yes" active="no"/>
-<layer number="53" name="tGND_GNDA" color="7" fill="9" visible="yes" active="no"/>
-<layer number="54" name="bGND_GNDA" color="1" fill="9" visible="yes" active="no"/>
-<layer number="56" name="wert" color="7" fill="1" visible="yes" active="no"/>
-<layer number="57" name="tCAD" color="7" fill="1" visible="yes" active="no"/>
+<layer number="46" name="Milling" color="3" fill="1" visible="no" active="no"/>
+<layer number="47" name="Measures" color="7" fill="1" visible="no" active="no"/>
+<layer number="48" name="Document" color="7" fill="1" visible="no" active="no"/>
+<layer number="49" name="Reference" color="7" fill="1" visible="no" active="no"/>
+<layer number="50" name="dxf" color="7" fill="1" visible="no" active="no"/>
+<layer number="51" name="tDocu" color="7" fill="1" visible="no" active="no"/>
+<layer number="52" name="bDocu" color="7" fill="1" visible="no" active="no"/>
+<layer number="53" name="tGND_GNDA" color="7" fill="9" visible="no" active="no"/>
+<layer number="54" name="bGND_GNDA" color="1" fill="9" visible="no" active="no"/>
+<layer number="56" name="wert" color="7" fill="1" visible="no" active="no"/>
+<layer number="57" name="tCAD" color="7" fill="1" visible="no" active="no"/>
 <layer number="90" name="Modules" color="5" fill="1" visible="yes" active="yes"/>
 <layer number="91" name="Nets" color="2" fill="1" visible="yes" active="yes"/>
@@
 </busses>
 <nets>
-<net name="GND" class="1">
+<net name="GND" class="0">
 <segment>
 <wire x1="251.46" y1="259.08" x2="256.54" y2="259.08" width="0.1524" layer="91"/>
@@
 </segment>
 </net>
-<net name="I2C1_SCL" class="0">
+<net name="N$11" class="0">
 <segment>
 <wire x1="162.56" y1="180.34" x2="139.7" y2="180.34" width="0.1524" layer="91"/>

Commit message: board update
Parts:
- R1, R2: device SparkFun-Passives:RESISTOR0402-RES -> SparkFun-Passives:RESISTOR0603-RES
Connections:
- net N$11 renamed I2C1_SCL
Changed lines of the file:
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@@
 <grid distance="0.1" unitdist="inch" unit="inch" style="lines" multiple="1" display="no" altdistance="0.01" altunitdist="inch" altunit="inch"/>
 <layers>
-<layer number="1" name="Top" color="4" fill="1" visible="no" active="no"/>
-<layer number="2" name="Route2" color="1" fill="3" visible="no" active="no"/>
-<layer number="3" name="Route3" color="4" fill="3" visible="no" active="no"/>
-<layer number="14" name="Route14" color="1" fill="6" visible="no" active="no"/>
-<layer number="15" name="Route15" color="4" fill="6" visible="no" active="no"/>
-<layer number="16" name="Bottom" color="1" fill="1" visible="no" active="no"/>
-<layer number="17" name="Pads" color="2" fill="1" visible="no" active="no"/>
-<layer number="18" name="Vias" color="2" fill="1" visible="no" active="no"/>
-<layer number="19" name="Unrouted" color="6" fill="1" visible="no" active="no"/>
-<layer number="20" name="Dimension" color="15" fill="1" visible="no" active="no"/>
-<layer number="21" name="tPlace" color="7" fill="1" visible="no" active="no"/>
-<layer number="22" name="bPlace" color="7" fill="1" visible="no" active="no"/>
-<layer number="23" name="tOrigins" color="15" fill="1" visible="no" active="no"/>
-<layer number="24" name="bOrigins" color="15" fill="1" visible="no" active="no"/>
-<layer number="25" name="tNames" color="7" fill="1" visible="no" active="no"/>
-<layer number="26" name="bNames" color="7" fill="1" visible="no" active="no"/>
-<layer number="27" name="tValues" color="7" fill="1" visible="no" active="no"/>
-<layer number="28" name="bValues" color="7" fill="1" visible="no" active="no"/>
+<layer number="1" name="Top" color="4" fill="1" visible="yes" active="no"/>
+<layer number="2" name="Route2" color="1" fill="3" visible="yes" active="no"/>
+<layer number="3" name="Route3" color="4" fill="3" visible="yes" active="no"/>
+<layer number="14" name="Route14" color="1" fill="6" visible="yes" active="no"/>
+<layer number="15" name="Route15" color="4" fill="6" visible="yes" active="no"/>
+<layer number="16" name="Bottom" color="1" fill="1" visible="yes" active="no"/>
+<layer number="17" name="Pads" color="2" fill="1" visible="yes" active="no"/>
+<layer number="18" name="Vias" color="2" fill="1" visible="yes" active="no"/>
+<layer number="19" name="Unrouted" color="6" fill="1" visible="yes" active="no"/>
+<layer number="20" name="Dimension" color="15" fill="1" visible="yes" active="no"/>
+<layer number="21" name="tPlace" color="7" fill="1" visible="yes" active="no"/>
+<layer number="22" name="bPlace" color="7" fill="1" visible="yes" active="no"/>
+<layer number="23" name="tOrigins" color="15" fill="1" visible="yes" active="no"/>
+<layer number="24" name="bOrigins" color="15" fill="1" visible="yes" active="no"/>
+<layer number="25" name="tNames" color="7" fill="1" visible="yes" active="no"/>
+<layer number="26" name="bNames" color="7" fill="1" visible="yes" active="no"/>
+<layer number="27" name="tValues" color="7" fill="1" visible="yes" active="no"/>
+<layer number="28" name="bValues" color="7" fill="1" visible="yes" active="no"/>
 <layer number="29" name="tStop" color="7" fill="3" visible="no" active="no"/>
 <layer number="30" name="bStop" color="7" fill="6" visible="no" active="no"/>
@@
 <layer number="35" name="tGlue" color="7" fill="4" visible="no" active="no"/>
 <layer number="36" name="bGlue" color="7" fill="5" visible="no" active="no"/>
-<layer number="37" name="tTest" color="7" fill="1" visible="no" active="no"/>
-<layer number="38" name="bTest" color="7" fill="1" visible="no" active="no"/>
+<layer number="37" name="tTest" color="7" fill="1" visible="yes" active="no"/>
+<layer number="38" name="bTest" color="7" fill="1" visible="yes" active="no"/>
 <layer number="39" name="tKeepout" color="4" fill="11" visible="no" active="no"/>
 <layer number="40" name="bKeepout" color="1" fill="11" visible="no" active="no"/>
@@
 <layer number="44" name="Drills" color="7" fill="1" visible="no" active="no"/>
 <layer number="45" name="Holes" color="7" fill="1" visible="no" active="no"/>
-<layer number="46" name="Milling" color="3" fill="1" visible="no" active="no"/>
-<layer number="47" name="Measures" color="7" fill="1" visible="no" active="no"/>
-<layer number="48" name="Document" color="7" fill="1" visible="no" active="no"/>
-<layer number="49" name="Reference" color="7" fill="1" visible="no" active="no"/>
-<layer number="50" name="dxf" color="7" fill="1" visible="no" active="no"/>
-<layer number="51" name="tDocu" color="7" fill="1" visible="no" active="no"/>
-<layer number="52" name="bDocu" color="7" fill="1" visible="no" active="no"/>
-<layer number="53" name="tGND_GNDA" color="7" fill="9" visible="no" active="no"/>
-<layer number="54" name="bGND_GNDA" color="1" fill="9" visible="no" active="no"/>
-<layer number="56" name="wert" color="7" fill="1" visible="no" active="no"/>
-<layer number="57" name="tCAD" color="7" fill="1" visible="no" active="no"/>
+<layer number="46" name="Milling" color="3" fill="1" visible="yes" active="no"/>
+<layer number="47" name="Measures" color="7" fill="1" visible="yes" active="no"/>
+<layer number="48" name="Document" color="7" fill="1" visible="yes" active="no"/>
+<layer number="49" name="Reference" color="7" fill="1" visible="yes" active="no"/>
+<layer number="50" name="dxf" color="7" fill="1" visible="yes" active="no"/>
+<layer number="51" name="tDocu" color="7" fill="1" visible="yes" active="no"/>
+<layer number="52" name="bDocu" color="7" fill="1" visible="yes" active="no"/>
+<layer number="53" name="tGND_GNDA" color="7" fill="9" visible="yes" active="no"/>
+<layer number="54" name="bGND_GNDA" color="1" fill="9" visible="yes" active="no"/>
+<layer number="56" name="wert" color="7" fill="1" visible="yes" active="no"/>
+<layer number="57" name="tCAD" color="7" fill="1" visible="yes" active="no"/>
 <layer number="90" name="Modules" color="5" fill="1" visible="yes" active="yes"/>
 <layer number="91" name="Nets" color="2" fill="1" visible="yes" active="yes"/>
@@
 <part name="C3" library="SparkFun-Capacitors" deviceset="CAP" device="0603-CAP" value="4.7uF"/>
 <part name="C1" library="SparkFun-Capacitors" deviceset="CAP" device="0603-CAP" value="10nF"/>
-<part name="R1" library="SparkFun-Passives" deviceset="RESISTOR" device="0402-RES" value="10k"/>
+<part name="R1" library="SparkFun-Passives" deviceset="RESISTOR" device="0603-RES" value="10k"/>
 <part name="SUPPLY1" library="SparkFun-Aesthetics" deviceset="VCC" device=""/>
-<part name="R2" library="SparkFun-Passives" deviceset="RESISTOR" device="0402-RES" value="10k"/>
+<part name="R2" library="SparkFun-Passives" deviceset="RESISTOR" device="0603-RES" value="10k"/>
 <part name="U2" library="Microchip_By_element14_Batch_1" deviceset="MCP1700T-3302E/TT" device=""/>
 <part name="U3" library="Microchip_By_element14_Batch_1" deviceset="MCP1700T-3302E/TT" device=""/>
@@
 <pinref part="U4" gate="G$1" pin="CS"/>
 <wire x1="388.62" y1="180.34" x2="388.62" y2="177.8" width="0.1524" layer="91"/>
-<wire x1="358.14" y1="177.8" x2="383.54" y2="177.8" width="0.1524" layer="91"/>
-<label x="360.68" y="177.8" size="1.778" layer="95"/>
-<wire x1="383.54" y1="177.8" x2="383.54" y2="180.34" width="0.1524" layer="91"/>
-<wire x1="383.54" y1="180.34" x2="388.62" y2="180.34" width="0.1524" layer="91"/>
+<wire x1="358.14" y1="177.8" x2="386.08" y2="177.8" width="0.1524" layer="91"/>
+<wire x1="386.08" y1="177.8" x2="386.08" y2="180.34" width="0.1524" layer="91"/>
+<wire x1="386.08" y1="180.34" x2="388.62" y2="180.34" width="0.1524" layer="91"/>
 <junction x="388.62" y="180.34"/>
 </segment>
@@
 </segment>
 </net>
-<net name="N$11" class="0">
+<net name="I2C1_SCL" class="0">
 <segment>
 <wire x1="162.56" y1="180.34" x2="139.7" y2="180.34" width="0.1524" layer="91"/>
@@
 <wire x1="302.26" y1="101.6" x2="302.26" y2="99.06" width="0.1524" layer="91"/>
 <junction x="302.26" y="99.06"/>
-<wire x1="309.88" y1="99.06" x2="314.96" y2="99.06" width="0.1524" layer="91"/>
-<label x="314.96" y="99.06" size="1.778" layer="95" xref="yes"/>
-</segment>
-<segment>
+</segment>
+<segment>
