File: PCB Design/STM32/stm32.sch (EAGLE design)
At the start: 68 parts, among them IC1 NCP1117ST50T3G, Q1 ABM3B-8.000MHZ-10-1UT, T5 BC847, T6 BC847, T7 BC847, T8 BC847, U1 STM32F103RET6, U2 MCP1700T-3302E/TT, U3 MCP1700T-3302E/TT, U4 MPU-6050, U5 TB6612FNG, X1 22-23-2031

Commit message: save
Parts:
- added R18, R20, R21, R23: (no value), SparkFun-Resistors:RESISTOR0805-RES
Connections:
- new net N$20: R18.2, U1.PB12
- new net N$21: R20.2, U1.PB13
- new net N$29: R21.2, U1.PB14
- new net N$30: R23.2, U1.PB15
- net M1CA: now also R18.1; no longer U1.PB12
- net M1CB: now also R20.1; no longer U1.PB13
- net M2CA: now also R23.1; no longer U1.PB15
- net M2CB: now also R21.1; no longer U1.PB14
Changed lines of the file:
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@@
 <part name="SUPPLY19" library="SparkFun-Aesthetics" deviceset="5V" device=""/>
 <part name="SUPPLY23" library="SparkFun-Aesthetics" deviceset="5V" device=""/>
+<part name="R18" library="SparkFun-Resistors" deviceset="RESISTOR" device="0805-RES"/>
+<part name="R20" library="SparkFun-Resistors" deviceset="RESISTOR" device="0805-RES"/>
+<part name="R21" library="SparkFun-Resistors" deviceset="RESISTOR" device="0805-RES"/>
+<part name="R23" library="SparkFun-Resistors" deviceset="RESISTOR" device="0805-RES"/>
 </parts>
 <sheets>
@@
 <instance part="SUPPLY19" gate="G$1" x="429.26" y="134.62"/>
 <instance part="SUPPLY23" gate="G$1" x="429.26" y="114.3"/>
+<instance part="R18" gate="G$1" x="149.86" y="165.1"/>
+<instance part="R20" gate="G$1" x="149.86" y="162.56"/>
+<instance part="R21" gate="G$1" x="149.86" y="160.02"/>
+<instance part="R23" gate="G$1" x="149.86" y="157.48"/>
 </instances>
 <busses>
@@
 <net name="M1CB" class="0">
 <segment>
-<wire x1="162.56" y1="162.56" x2="147.32" y2="162.56" width="0.1524" layer="91"/>
-<label x="154.94" y="162.56" size="1.778" layer="95" rot="MR0"/>
-<pinref part="U1" gate="A" pin="PB13"/>
-</segment>
-<segment>
 <pinref part="JP4" gate="G$1" pin="5"/>
 <wire x1="401.32" y1="109.22" x2="393.7" y2="109.22" width="0.1524" layer="91"/>
 <label x="393.7" y="106.68" size="1.778" layer="95"/>
 </segment>
+<segment>
+<pinref part="R20" gate="G$1" pin="1"/>
+<wire x1="144.78" y1="162.56" x2="139.7" y2="162.56" width="0.1524" layer="91"/>
+<label x="137.16" y="162.56" size="1.778" layer="95"/>
+</segment>
 </net>
 <net name="M1CA" class="0">
-<segment>
-<wire x1="162.56" y1="165.1" x2="147.32" y2="165.1" width="0.1524" layer="91"/>
-<label x="154.94" y="165.1" size="1.778" layer="95" rot="MR0"/>
-<pinref part="U1" gate="A" pin="PB12"/>
-</segment>
 <segment>
 <pinref part="JP4" gate="G$1" pin="6"/>
@@
 <label x="419.1" y="106.68" size="1.778" layer="95"/>
 </segment>
+<segment>
+<pinref part="R18" gate="G$1" pin="1"/>
+<wire x1="144.78" y1="165.1" x2="139.7" y2="165.1" width="0.1524" layer="91"/>
+<label x="137.16" y="165.1" size="1.778" layer="95"/>
+</segment>
 </net>
 <net name="M2CA" class="0">
@@
 </segment>
 <segment>
-<wire x1="162.56" y1="157.48" x2="147.32" y2="157.48" width="0.1524" layer="91"/>
-<label x="154.94" y="157.48" size="1.778" layer="95" rot="MR0"/>
-<pinref part="U1" gate="A" pin="PB15"/>
+<pinref part="R23" gate="G$1" pin="1"/>
+<wire x1="144.78" y1="157.48" x2="139.7" y2="157.48" width="0.1524" layer="91"/>
+<label x="137.16" y="157.48" size="1.778" layer="95"/>
 </segment>
 </net>
@@
 </segment>
 <segment>
-<wire x1="162.56" y1="160.02" x2="147.32" y2="160.02" width="0.1524" layer="91"/>
-<label x="154.94" y="160.02" size="1.778" layer="95" rot="MR0"/>
-<pinref part="U1" gate="A" pin="PB14"/>
+<pinref part="R21" gate="G$1" pin="1"/>
+<wire x1="144.78" y1="160.02" x2="139.7" y2="160.02" width="0.1524" layer="91"/>
+<label x="137.16" y="160.02" size="1.778" layer="95"/>
 </segment>
 </net>
@@
 </segment>
 </net>
+<net name="N$20" class="0">
+<segment>
+<pinref part="R18" gate="G$1" pin="2"/>
+<pinref part="U1" gate="A" pin="PB12"/>
+<wire x1="154.94" y1="165.1" x2="162.56" y2="165.1" width="0.1524" layer="91"/>
+</segment>
+</net>
+<net name="N$21" class="0">
+<segment>
+<pinref part="R20" gate="G$1" pin="2"/>
+<pinref part="U1" gate="A" pin="PB13"/>
+<wire x1="154.94" y1="162.56" x2="162.56" y2="162.56" width="0.1524" layer="91"/>
+</segment>
+</net>
+<net name="N$29" class="0">
+<segment>
+<pinref part="R21" gate="G$1" pin="2"/>
+<pinref part="U1" gate="A" pin="PB14"/>
+<wire x1="154.94" y1="160.02" x2="162.56" y2="160.02" width="0.1524" layer="91"/>
+</segment>
+</net>
+<net name="N$30" class="0">
+<segment>
+<pinref part="R23" gate="G$1" pin="2"/>
+<pinref part="U1" gate="A" pin="PB15"/>
+<wire x1="154.94" y1="157.48" x2="162.56" y2="157.48" width="0.1524" layer="91"/>
+</segment>
+</net>

Commit message: sleep
Parts:
- removed R18, R20, R21, R23: (no value), SparkFun-Resistors:RESISTOR0805-RES
Connections:
- removed net N$20: R18.2, U1.PB12
- removed net N$21: R20.2, U1.PB13
- removed net N$29: R21.2, U1.PB14
- removed net N$30: R23.2, U1.PB15
- net M1CA: now also U1.PB12; no longer R18.1
- net M1CB: now also U1.PB13; no longer R20.1
- net M2CA: now also U1.PB15; no longer R23.1
- net M2CB: now also U1.PB14; no longer R21.1
Changed lines of the file:
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@@
 <part name="SUPPLY19" library="SparkFun-Aesthetics" deviceset="5V" device=""/>
 <part name="SUPPLY23" library="SparkFun-Aesthetics" deviceset="5V" device=""/>
-<part name="R18" library="SparkFun-Resistors" deviceset="RESISTOR" device="0805-RES"/>
-<part name="R20" library="SparkFun-Resistors" deviceset="RESISTOR" device="0805-RES"/>
-<part name="R21" library="SparkFun-Resistors" deviceset="RESISTOR" device="0805-RES"/>
-<part name="R23" library="SparkFun-Resistors" deviceset="RESISTOR" device="0805-RES"/>
 </parts>
 <sheets>
@@
 <instance part="SUPPLY19" gate="G$1" x="429.26" y="134.62"/>
 <instance part="SUPPLY23" gate="G$1" x="429.26" y="114.3"/>
-<instance part="R18" gate="G$1" x="149.86" y="165.1"/>
-<instance part="R20" gate="G$1" x="149.86" y="162.56"/>
-<instance part="R21" gate="G$1" x="149.86" y="160.02"/>
-<instance part="R23" gate="G$1" x="149.86" y="157.48"/>
 </instances>
 <busses>
@@
 </segment>
 <segment>
-<pinref part="R20" gate="G$1" pin="1"/>
-<wire x1="144.78" y1="162.56" x2="139.7" y2="162.56" width="0.1524" layer="91"/>
-<label x="137.16" y="162.56" size="1.778" layer="95"/>
+<wire x1="162.56" y1="162.56" x2="149.86" y2="162.56" width="0.1524" layer="91"/>
+<label x="149.86" y="162.56" size="1.778" layer="95"/>
+<pinref part="U1" gate="A" pin="PB13"/>
 </segment>
 </net>
@@
 </segment>
 <segment>
-<pinref part="R18" gate="G$1" pin="1"/>
-<wire x1="144.78" y1="165.1" x2="139.7" y2="165.1" width="0.1524" layer="91"/>
-<label x="137.16" y="165.1" size="1.778" layer="95"/>
+<wire x1="162.56" y1="165.1" x2="149.86" y2="165.1" width="0.1524" layer="91"/>
+<label x="149.86" y="165.1" size="1.778" layer="95"/>
+<pinref part="U1" gate="A" pin="PB12"/>
 </segment>
 </net>
@@
 </segment>
 <segment>
-<pinref part="R23" gate="G$1" pin="1"/>
-<wire x1="144.78" y1="157.48" x2="139.7" y2="157.48" width="0.1524" layer="91"/>
-<label x="137.16" y="157.48" size="1.778" layer="95"/>
+<wire x1="162.56" y1="157.48" x2="149.86" y2="157.48" width="0.1524" layer="91"/>
+<label x="149.86" y="157.48" size="1.778" layer="95"/>
+<pinref part="U1" gate="A" pin="PB15"/>
 </segment>
 </net>
@@
 </segment>
 <segment>
-<pinref part="R21" gate="G$1" pin="1"/>
-<wire x1="144.78" y1="160.02" x2="139.7" y2="160.02" width="0.1524" layer="91"/>
-<label x="137.16" y="160.02" size="1.778" layer="95"/>
+<wire x1="162.56" y1="160.02" x2="149.86" y2="160.02" width="0.1524" layer="91"/>
+<label x="149.86" y="160.02" size="1.778" layer="95"/>
+<pinref part="U1" gate="A" pin="PB14"/>
 </segment>
 </net>
@@
 </segment>
 </net>
-<net name="N$20" class="0">
-<segment>
-<pinref part="R18" gate="G$1" pin="2"/>
-<pinref part="U1" gate="A" pin="PB12"/>
-<wire x1="154.94" y1="165.1" x2="162.56" y2="165.1" width="0.1524" layer="91"/>
-</segment>
-</net>
-<net name="N$21" class="0">
-<segment>
-<pinref part="R20" gate="G$1" pin="2"/>
-<pinref part="U1" gate="A" pin="PB13"/>
-<wire x1="154.94" y1="162.56" x2="162.56" y2="162.56" width="0.1524" layer="91"/>
-</segment>
-</net>
-<net name="N$29" class="0">
-<segment>
-<pinref part="R21" gate="G$1" pin="2"/>
-<pinref part="U1" gate="A" pin="PB14"/>
-<wire x1="154.94" y1="160.02" x2="162.56" y2="160.02" width="0.1524" layer="91"/>
-</segment>
-</net>
-<net name="N$30" class="0">
-<segment>
-<pinref part="R23" gate="G$1" pin="2"/>
-<pinref part="U1" gate="A" pin="PB15"/>
-<wire x1="154.94" y1="157.48" x2="162.56" y2="157.48" width="0.1524" layer="91"/>
-</segment>
-</net>

Commit message: save
Connections:
- net JTAG-TCK: now also U$1.7; no longer U$1.5
- net JTAG-TDO: now also U$1.5; no longer U$1.7
Changed lines of the file:
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@@
 </segment>
 <segment>
-<wire x1="83.82" y1="172.72" x2="73.66" y2="172.72" width="0.1524" layer="91"/>
-<label x="83.82" y="172.72" size="1.778" layer="95" rot="MR0"/>
-<pinref part="U$1" gate="G$1" pin="5"/>
+<wire x1="83.82" y1="170.18" x2="73.66" y2="170.18" width="0.1524" layer="91"/>
+<label x="83.82" y="170.18" size="1.778" layer="95" rot="MR0"/>
+<pinref part="U$1" gate="G$1" pin="7"/>
 </segment>
 </net>
@@
 </segment>
 <segment>
-<wire x1="83.82" y1="170.18" x2="73.66" y2="170.18" width="0.1524" layer="91"/>
-<label x="83.82" y="170.18" size="1.778" layer="95" rot="MR0"/>
-<pinref part="U$1" gate="G$1" pin="7"/>
+<wire x1="83.82" y1="172.72" x2="73.66" y2="172.72" width="0.1524" layer="91"/>
+<label x="83.82" y="172.72" size="1.778" layer="95" rot="MR0"/>
+<pinref part="U$1" gate="G$1" pin="5"/>
 </segment>
 </net>
@@
 <pinref part="R7" gate="G$1" pin="2"/>
 <wire x1="365.76" y1="220.98" x2="365.76" y2="226.06" width="0.1524" layer="91"/>
-<wire x1="365.76" y1="226.06" x2="365.76" y2="228.346" width="0.1524" layer="91"/>
-<wire x1="365.76" y1="228.346" x2="365.76" y2="228.6" width="0.1524" layer="91"/>
 <wire x1="365.76" y1="226.06" x2="355.6" y2="226.06" width="0.1524" layer="91"/>
-<label x="358.14" y="226.06" size="1.778" layer="95"/>
+<label x="355.6" y="226.06" size="1.778" layer="95"/>
+<wire x1="365.76" y1="228.6" x2="365.76" y2="228.346" width="0.1524" layer="91"/>
 <junction x="365.76" y="226.06"/>
 <pinref part="U$2" gate="G$1" pin="P$E"/>
+<wire x1="365.76" y1="228.346" x2="365.76" y2="226.06" width="0.1524" layer="91"/>
 <junction x="365.76" y="228.346"/>
 </segment>
@@
 <pinref part="R8" gate="G$1" pin="2"/>
 <wire x1="386.08" y1="220.98" x2="386.08" y2="226.06" width="0.1524" layer="91"/>
-<wire x1="386.08" y1="226.06" x2="386.08" y2="228.346" width="0.1524" layer="91"/>
-<wire x1="386.08" y1="228.346" x2="386.08" y2="228.6" width="0.1524" layer="91"/>
 <wire x1="375.92" y1="226.06" x2="386.08" y2="226.06" width="0.1524" layer="91"/>
 <label x="375.92" y="226.06" size="1.778" layer="95"/>
+<wire x1="386.08" y1="228.6" x2="386.08" y2="228.346" width="0.1524" layer="91"/>
 <junction x="386.08" y="226.06"/>
 <pinref part="U$3" gate="G$1" pin="P$E"/>
+<wire x1="386.08" y1="228.346" x2="386.08" y2="226.06" width="0.1524" layer="91"/>
 <junction x="386.08" y="228.346"/>
 </segment>
@@
 <pinref part="R9" gate="G$1" pin="2"/>
 <wire x1="406.4" y1="220.98" x2="406.4" y2="226.06" width="0.1524" layer="91"/>
-<wire x1="406.4" y1="226.06" x2="406.4" y2="228.346" width="0.1524" layer="91"/>
-<wire x1="406.4" y1="228.346" x2="406.4" y2="228.6" width="0.1524" layer="91"/>
 <wire x1="396.24" y1="226.06" x2="406.4" y2="226.06" width="0.1524" layer="91"/>
 <label x="396.24" y="226.06" size="1.778" layer="95"/>
+<wire x1="406.4" y1="228.6" x2="406.4" y2="228.346" width="0.1524" layer="91"/>
 <junction x="406.4" y="226.06"/>
 <pinref part="U$4" gate="G$1" pin="P$E"/>
+<wire x1="406.4" y1="228.346" x2="406.4" y2="226.06" width="0.1524" layer="91"/>
 <junction x="406.4" y="228.346"/>
 </segment>
@@
 </segment>
 <segment>
-<pinref part="R10" gate="G$1" pin="2"/>
-<wire x1="429.26" y1="220.98" x2="429.26" y2="226.06" width="0.1524" layer="91"/>
-<wire x1="429.26" y1="226.06" x2="429.26" y2="228.346" width="0.1524" layer="91"/>
-<wire x1="429.26" y1="228.346" x2="429.26" y2="228.6" width="0.1524" layer="91"/>
 <wire x1="419.1" y1="226.06" x2="429.26" y2="226.06" width="0.1524" layer="91"/>
 <label x="419.1" y="226.06" size="1.778" layer="95"/>
+<pinref part="R10" gate="G$1" pin="2"/>
+<wire x1="429.26" y1="228.6" x2="429.26" y2="228.346" width="0.1524" layer="91"/>
 <junction x="429.26" y="226.06"/>
+<wire x1="429.26" y1="228.346" x2="429.26" y2="226.06" width="0.1524" layer="91"/>
+<wire x1="429.26" y1="226.06" x2="429.26" y2="220.98" width="0.1524" layer="91"/>
 <pinref part="U$5" gate="G$1" pin="P$E"/>
 <junction x="429.26" y="228.346"/>

Commit message: save
Connections:
- removed net LED4: U1.PB1
Changed lines of the file:
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@@
 <pinref part="C13" gate="G$1" pin="1"/>
 <wire x1="243.84" y1="248.92" x2="251.46" y2="248.92" width="0.1524" layer="91"/>
+<junction x="251.46" y="248.92"/>
 </segment>
 <segment>
@@
 </segment>
 </net>
-<net name="LED4" class="0">
-<segment>
-<pinref part="U1" gate="A" pin="PB1"/>
-<wire x1="162.56" y1="190.5" x2="147.32" y2="190.5" width="0.1524" layer="91"/>
-<label x="147.32" y="190.5" size="1.778" layer="95"/>
-</segment>
-</net>

Commit message: ultimate final edition
Parts:
- LED5, LED6, LED7: device eagle-ltspice:LED_ESML0603 -> led:LEDSML0805
Changed lines of the file:
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@@
 <part name="R13" library="SparkFun-Resistors" deviceset="RESISTOR" device="0805-RES" value="2k"/>
 <part name="R14" library="SparkFun-Resistors" deviceset="RESISTOR" device="0805-RES" value="2k"/>
-<part name="LED5" library="eagle-ltspice" deviceset="LED_E" device="SML0603"/>
-<part name="LED6" library="eagle-ltspice" deviceset="LED_E" device="SML0603"/>
-<part name="LED7" library="eagle-ltspice" deviceset="LED_E" device="SML0603"/>
+<part name="LED5" library="led" deviceset="LED" device="SML0805"/>
+<part name="LED6" library="led" deviceset="LED" device="SML0805"/>
+<part name="LED7" library="led" deviceset="LED" device="SML0805"/>
 <part name="R15" library="SparkFun-Resistors" deviceset="RESISTOR" device="0805-RES"/>
 <part name="R16" library="SparkFun-Resistors" deviceset="RESISTOR" device="0805-RES"/>

Commit message: emergency update
Connections:
- net I2C1_SCL: now also U1.PB8; no longer U1.PB6
- net I2C1_SDA: now also U1.PB9; no longer U1.PB7
- net INT: no longer U1.PB8
- net IR_OUT1: now also U1.PB12; no longer U1.PC9
- net IR_OUT2: now also U1.PB13; no longer U1.PC8
- net IR_OUT3: now also U1.PB14; no longer U1.PC7
- net IR_OUT4: now also U1.PB15; no longer U1.PC6
- net M1CA: now also U1.PB6; no longer U1.PB12
- net M1CB: now also U1.PB7; no longer U1.PB13
- net M2CA: now also U1.PC6; no longer U1.PB15
- net M2CB: now also U1.PC7; no longer U1.PB14
Other:
- moved on the sheet: R1, R2
Changed lines of the file:
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@@
 <instance part="C3" gate="G$1" x="83.82" y="215.9"/>
 <instance part="C1" gate="G$1" x="99.06" y="251.46"/>
-<instance part="R1" gate="G$1" x="134.62" y="180.34" rot="MR0"/>
-<instance part="SUPPLY1" gate="G$1" x="124.46" y="182.88" rot="MR0"/>
-<instance part="R2" gate="G$1" x="134.62" y="172.72" rot="MR0"/>
+<instance part="R1" gate="G$1" x="134.62" y="175.26" rot="MR0"/>
+<instance part="SUPPLY1" gate="G$1" x="124.46" y="177.8" rot="MR0"/>
+<instance part="R2" gate="G$1" x="134.62" y="167.64" rot="MR0"/>
 <instance part="U2" gate="A" x="210.82" y="111.76"/>
 <instance part="U3" gate="A" x="210.82" y="83.82"/>
@@
 <segment>
 <pinref part="SUPPLY1" gate="G$1" pin="VCC"/>
-<wire x1="124.46" y1="182.88" x2="124.46" y2="180.34" width="0.1524" layer="91"/>
+<wire x1="124.46" y1="177.8" x2="124.46" y2="175.26" width="0.1524" layer="91"/>
 <pinref part="R1" gate="G$1" pin="2"/>
-<wire x1="129.54" y1="180.34" x2="127" y2="180.34" width="0.1524" layer="91"/>
-<wire x1="127" y1="180.34" x2="127" y2="172.72" width="0.1524" layer="91"/>
+<wire x1="129.54" y1="175.26" x2="127" y2="175.26" width="0.1524" layer="91"/>
+<wire x1="127" y1="175.26" x2="127" y2="167.64" width="0.1524" layer="91"/>
 <pinref part="R2" gate="G$1" pin="2"/>
-<wire x1="127" y1="172.72" x2="129.54" y2="172.72" width="0.1524" layer="91"/>
-<wire x1="124.46" y1="180.34" x2="127" y2="180.34" width="0.1524" layer="91"/>
-<junction x="127" y="180.34"/>
+<wire x1="127" y1="167.64" x2="129.54" y2="167.64" width="0.1524" layer="91"/>
+<wire x1="124.46" y1="175.26" x2="127" y2="175.26" width="0.1524" layer="91"/>
+<junction x="127" y="175.26"/>
 </segment>
 <segment>
@@
 <net name="I2C1_SDA" class="0">
 <segment>
-<wire x1="162.56" y1="177.8" x2="142.24" y2="177.8" width="0.1524" layer="91"/>
-<label x="147.32" y="177.8" size="1.778" layer="95"/>
-<wire x1="142.24" y1="177.8" x2="142.24" y2="172.72" width="0.1524" layer="91"/>
-<wire x1="142.24" y1="172.72" x2="139.7" y2="172.72" width="0.1524" layer="91"/>
+<wire x1="142.24" y1="172.72" x2="142.24" y2="167.64" width="0.1524" layer="91"/>
+<wire x1="142.24" y1="167.64" x2="139.7" y2="167.64" width="0.1524" layer="91"/>
 <pinref part="R2" gate="G$1" pin="1"/>
-<pinref part="U1" gate="A" pin="PB7"/>
+<pinref part="U1" gate="A" pin="PB9"/>
+<wire x1="142.24" y1="172.72" x2="162.56" y2="172.72" width="0.1524" layer="91"/>
+<label x="147.32" y="172.72" size="1.778" layer="95"/>
 </segment>
 <segment>
@@
 <net name="I2C1_SCL" class="0">
 <segment>
-<wire x1="162.56" y1="180.34" x2="139.7" y2="180.34" width="0.1524" layer="91"/>
-<label x="147.32" y="180.34" size="1.778" layer="95"/>
-<pinref part="R1" gate="G$1" pin="1"/>
-<pinref part="U1" gate="A" pin="PB6"/>
-</segment>
-<segment>
 <pinref part="U4" gate="G$1" pin="SCL/SCLK"/>
 <wire x1="358.14" y1="175.26" x2="365.76" y2="175.26" width="0.1524" layer="91"/>
 <label x="360.68" y="175.26" size="1.778" layer="95"/>
+</segment>
+<segment>
+<pinref part="U1" gate="A" pin="PB8"/>
+<pinref part="R1" gate="G$1" pin="1"/>
+<wire x1="162.56" y1="175.26" x2="139.7" y2="175.26" width="0.1524" layer="91"/>
+<label x="147.32" y="175.26" size="1.778" layer="95"/>
 </segment>
 </net>
@@
 </segment>
 <segment>
-<pinref part="U1" gate="A" pin="PC8"/>
-<wire x1="223.52" y1="226.06" x2="238.76" y2="226.06" width="0.1524" layer="91"/>
-<label x="228.6" y="226.06" size="1.778" layer="95"/>
+<pinref part="U1" gate="A" pin="PB13"/>
+<wire x1="162.56" y1="162.56" x2="147.32" y2="162.56" width="0.1524" layer="91"/>
+<label x="147.32" y="162.56" size="1.778" layer="95"/>
 </segment>
 </net>
@@
 </segment>
 <segment>
-<pinref part="U1" gate="A" pin="PC9"/>
-<wire x1="223.52" y1="223.52" x2="238.76" y2="223.52" width="0.1524" layer="91"/>
-<label x="228.6" y="223.52" size="1.778" layer="95"/>
+<pinref part="U1" gate="A" pin="PB12"/>
+<wire x1="162.56" y1="165.1" x2="147.32" y2="165.1" width="0.1524" layer="91"/>
+<label x="147.32" y="165.1" size="1.778" layer="95"/>
 </segment>
 </net>
@@
 </segment>
 <segment>
-<pinref part="U1" gate="A" pin="PC7"/>
-<wire x1="223.52" y1="228.6" x2="238.76" y2="228.6" width="0.1524" layer="91"/>
-<label x="228.6" y="228.6" size="1.778" layer="95"/>
+<pinref part="U1" gate="A" pin="PB14"/>
+<wire x1="162.56" y1="160.02" x2="147.32" y2="160.02" width="0.1524" layer="91"/>
+<label x="147.32" y="160.02" size="1.778" layer="95"/>
 </segment>
 </net>
@@
 </segment>
 <segment>
-<pinref part="U1" gate="A" pin="PC6"/>
-<wire x1="223.52" y1="231.14" x2="238.76" y2="231.14" width="0.1524" layer="91"/>
-<label x="228.6" y="231.14" size="1.778" layer="95"/>
+<pinref part="U1" gate="A" pin="PB15"/>
+<wire x1="162.56" y1="157.48" x2="147.32" y2="157.48" width="0.1524" layer="91"/>
+<label x="147.32" y="157.48" size="1.778" layer="95"/>
 </segment>
 </net>
@@
 <wire x1="322.58" y1="175.26" x2="314.96" y2="175.26" width="0.1524" layer="91"/>
 <label x="314.96" y="175.26" size="1.778" layer="95"/>
-</segment>
-<segment>
-<wire x1="162.56" y1="175.26" x2="147.32" y2="175.26" width="0.1524" layer="91"/>
-<label x="147.32" y="175.26" size="1.778" layer="95"/>
-<pinref part="U1" gate="A" pin="PB8"/>
 </segment>
 </net>
@@
 </segment>
 <segment>
-<wire x1="162.56" y1="162.56" x2="149.86" y2="162.56" width="0.1524" layer="91"/>
-<label x="149.86" y="162.56" size="1.778" layer="95"/>
-<pinref part="U1" gate="A" pin="PB13"/>
+<pinref part="U1" gate="A" pin="PB7"/>
+<wire x1="162.56" y1="177.8" x2="147.32" y2="177.8" width="0.1524" layer="91"/>
+<label x="147.32" y="177.8" size="1.778" layer="95"/>
 </segment>
 </net>
@@
 </segment>
 <segment>
-<wire x1="162.56" y1="165.1" x2="149.86" y2="165.1" width="0.1524" layer="91"/>
-<label x="149.86" y="165.1" size="1.778" layer="95"/>
-<pinref part="U1" gate="A" pin="PB12"/>
+<pinref part="U1" gate="A" pin="PB6"/>
+<wire x1="162.56" y1="180.34" x2="147.32" y2="180.34" width="0.1524" layer="91"/>
+<label x="147.32" y="180.34" size="1.778" layer="95"/>
 </segment>
 </net>
@@
 </segment>
 <segment>
-<wire x1="162.56" y1="157.48" x2="149.86" y2="157.48" width="0.1524" layer="91"/>
-<label x="149.86" y="157.48" size="1.778" layer="95"/>
-<pinref part="U1" gate="A" pin="PB15"/>
+<pinref part="U1" gate="A" pin="PC6"/>
+<wire x1="223.52" y1="231.14" x2="238.76" y2="231.14" width="0.1524" layer="91"/>
+<label x="228.6" y="231.14" size="1.778" layer="95"/>
 </segment>
 </net>
@@
 </segment>
 <segment>
-<wire x1="162.56" y1="160.02" x2="149.86" y2="160.02" width="0.1524" layer="91"/>
-<label x="149.86" y="160.02" size="1.778" layer="95"/>
-<pinref part="U1" gate="A" pin="PB14"/>
-</segment>
-</net>
+<pinref part="U1" gate="A" pin="PC7"/>
+<wire x1="223.52" y1="228.6" x2="238.76" y2="228.6" width="0.1524" layer="91"/>
+<label x="228.6" y="228.6" size="1.778" layer="95"/>
+</segment>
+</net>
