File: PCB Design/STM32/stm32.sch (EAGLE design)
At the start: 68 parts, among them IC1 NCP1117ST50T3G, Q1 ABM3B-8.000MHZ-10-1UT, T5 BC847, T6 BC847, T7 BC847, T8 BC847, U1 STM32F103RET6, U2 MCP1700T-3302E/TT, U3 MCP1700T-3302E/TT, U4 MPU-6050, U5 TB6612FNG, X1 22-23-2031

Commit message: finish update
Connections:
- net INT: now also U1.PC12
- net IR_OUT1: now also U1.PB15; no longer U1.PB12
- net IR_OUT2: now also U1.PB14; no longer U1.PB13
- net IR_OUT3: now also U1.PB13; no longer U1.PB14
- net IR_OUT4: now also U1.PB12; no longer U1.PB15
- net M1CA: now also U1.PB7; no longer U1.PB6
- net M1CB: now also U1.PB6; no longer U1.PB7
- net M2CA: now also U1.PC7; no longer U1.PC6
- net M2CB: now also U1.PC6; no longer U1.PC7
Changed lines of the file:
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@@
+</segment>
+<segment>
+<pinref part="U1" gate="A" pin="PB14"/>
+<wire x1="162.56" y1="160.02" x2="147.32" y2="160.02" width="0.1524" layer="91"/>
+<label x="147.32" y="160.02" size="1.778" layer="95"/>
+</segment>
+</net>
+<net name="IR_OUT1" class="0">
+<segment>
+<pinref part="R11" gate="G$1" pin="2"/>
+<wire x1="259.08" y1="236.22" x2="259.08" y2="226.06" width="0.1524" layer="91"/>
+<label x="259.08" y="228.6" size="1.778" layer="95"/>
+</segment>
+<segment>
+<pinref part="U1" gate="A" pin="PB15"/>
+<wire x1="162.56" y1="157.48" x2="147.32" y2="157.48" width="0.1524" layer="91"/>
+<label x="147.32" y="157.48" size="1.778" layer="95"/>
+</segment>
+</net>
+<net name="IR_OUT3" class="0">
+<segment>
+<pinref part="R13" gate="G$1" pin="2"/>
+<wire x1="304.8" y1="236.22" x2="304.8" y2="226.06" width="0.1524" layer="91"/>
+<label x="304.8" y="228.6" size="1.778" layer="95"/>
 </segment>
 <segment>
@@
 <wire x1="162.56" y1="162.56" x2="147.32" y2="162.56" width="0.1524" layer="91"/>
 <label x="147.32" y="162.56" size="1.778" layer="95"/>
-</segment>
-</net>
-<net name="IR_OUT1" class="0">
-<segment>
-<pinref part="R11" gate="G$1" pin="2"/>
-<wire x1="259.08" y1="236.22" x2="259.08" y2="226.06" width="0.1524" layer="91"/>
-<label x="259.08" y="228.6" size="1.778" layer="95"/>
-</segment>
-<segment>
-<pinref part="U1" gate="A" pin="PB12"/>
-<wire x1="162.56" y1="165.1" x2="147.32" y2="165.1" width="0.1524" layer="91"/>
-<label x="147.32" y="165.1" size="1.778" layer="95"/>
-</segment>
-</net>
-<net name="IR_OUT3" class="0">
-<segment>
-<pinref part="R13" gate="G$1" pin="2"/>
-<wire x1="304.8" y1="236.22" x2="304.8" y2="226.06" width="0.1524" layer="91"/>
-<label x="304.8" y="228.6" size="1.778" layer="95"/>
-</segment>
-<segment>
-<pinref part="U1" gate="A" pin="PB14"/>
-<wire x1="162.56" y1="160.02" x2="147.32" y2="160.02" width="0.1524" layer="91"/>
-<label x="147.32" y="160.02" size="1.778" layer="95"/>
 </segment>
 </net>
@@
 </segment>
 <segment>
-<pinref part="U1" gate="A" pin="PB15"/>
-<wire x1="162.56" y1="157.48" x2="147.32" y2="157.48" width="0.1524" layer="91"/>
-<label x="147.32" y="157.48" size="1.778" layer="95"/>
+<pinref part="U1" gate="A" pin="PB12"/>
+<wire x1="162.56" y1="165.1" x2="147.32" y2="165.1" width="0.1524" layer="91"/>
+<label x="147.32" y="165.1" size="1.778" layer="95"/>
 </segment>
 </net>
@@
 <wire x1="322.58" y1="175.26" x2="314.96" y2="175.26" width="0.1524" layer="91"/>
 <label x="314.96" y="175.26" size="1.778" layer="95"/>
+</segment>
+<segment>
+<pinref part="U1" gate="A" pin="PC12"/>
+<wire x1="223.52" y1="215.9" x2="238.76" y2="215.9" width="0.1524" layer="91"/>
+<label x="228.6" y="215.9" size="1.778" layer="95"/>
 </segment>
 </net>
@@
 </segment>
 <segment>
+<pinref part="U1" gate="A" pin="PB6"/>
+<wire x1="162.56" y1="180.34" x2="147.32" y2="180.34" width="0.1524" layer="91"/>
+<label x="147.32" y="180.34" size="1.778" layer="95"/>
+</segment>
+</net>
+<net name="M1CA" class="0">
+<segment>
+<pinref part="JP4" gate="G$1" pin="6"/>
+<wire x1="416.56" y1="109.22" x2="424.18" y2="109.22" width="0.1524" layer="91"/>
+<label x="419.1" y="106.68" size="1.778" layer="95"/>
+</segment>
+<segment>
 <pinref part="U1" gate="A" pin="PB7"/>
 <wire x1="162.56" y1="177.8" x2="147.32" y2="177.8" width="0.1524" layer="91"/>
@@
 </segment>
 </net>
-<net name="M1CA" class="0">
-<segment>
-<pinref part="JP4" gate="G$1" pin="6"/>
-<wire x1="416.56" y1="109.22" x2="424.18" y2="109.22" width="0.1524" layer="91"/>
-<label x="419.1" y="106.68" size="1.778" layer="95"/>
-</segment>
-<segment>
-<pinref part="U1" gate="A" pin="PB6"/>
-<wire x1="162.56" y1="180.34" x2="147.32" y2="180.34" width="0.1524" layer="91"/>
-<label x="147.32" y="180.34" size="1.778" layer="95"/>
-</segment>
-</net>
 <net name="M2CA" class="0">
 <segment>
@@
 </segment>
 <segment>
+<pinref part="U1" gate="A" pin="PC7"/>
+<wire x1="223.52" y1="228.6" x2="238.76" y2="228.6" width="0.1524" layer="91"/>
+<label x="228.6" y="228.6" size="1.778" layer="95"/>
+</segment>
+</net>
+<net name="M2CB" class="0">
+<segment>
+<pinref part="JP3" gate="G$1" pin="5"/>
+<wire x1="401.32" y1="129.54" x2="393.7" y2="129.54" width="0.1524" layer="91"/>
+<label x="393.7" y="127" size="1.778" layer="95"/>
+</segment>
+<segment>
 <pinref part="U1" gate="A" pin="PC6"/>
 <wire x1="223.52" y1="231.14" x2="238.76" y2="231.14" width="0.1524" layer="91"/>
@@
 </segment>
 </net>
-<net name="M2CB" class="0">
-<segment>
-<pinref part="JP3" gate="G$1" pin="5"/>
-<wire x1="401.32" y1="129.54" x2="393.7" y2="129.54" width="0.1524" layer="91"/>
-<label x="393.7" y="127" size="1.778" layer="95"/>
-</segment>
-<segment>
-<pinref part="U1" gate="A" pin="PC7"/>
-<wire x1="223.52" y1="228.6" x2="238.76" y2="228.6" width="0.1524" layer="91"/>
-<label x="228.6" y="228.6" size="1.778" layer="95"/>
-</segment>
-</net>
