File: PCB Design/STM32/stm32.brd (EAGLE design)
At the start: 48.8 x 69.3 mm, 72 parts, among them IC1 NCP1117ST50T3G, Q1 8MHz, T1 SFH303, T2 SFH303, T3 SFH303, T4 SFH303, U1 STM32F103RET6, U2 MCP1700T-3302E/TT, U3 MCP1700T-3302E/TT, U4 MPU-6050, U5 TB6612FNG

Commit message: meet update 1
Parts:
- C1, C12, C13, C16, C17, C18, C19, C20, C21, C3, C4, C5, C6, C7: device SparkFun-Capacitors:0603-CAP -> SparkFun-Capacitors:0805
- C10, C11: value 22uF -> 10uF; device rcl:UD-4X5,8_NICHICON -> SparkFun-Capacitors:0805
- C9: value 22uF -> 20uF; device rcl:UD-4X5,8_NICHICON -> SparkFun-Capacitors:0805
- R1, R2: device SparkFun-Passives:0603-RES -> SparkFun-Passives:0805
- R10: device resistor:R0603 -> SparkFun-Resistors:0805
- moved C11 4.78 mm to (48.3, 44.6)
- moved T2 3.92 mm to (57.7, 59.2)
- moved T1 1.55 mm to (48.3, 53.8)
- moved C10 1.42 mm to (52.3, 40.5), turned to 0 degrees
- moved C9 1.15 mm to (45.7, 43.6), turned to 90 degrees
- moved LED1 0.13 mm to (40.6, 48.8)
Connections:
- net 5V: now also C9.1; no longer C9.+
- net GND: now also C10.2, C11.2, C9.2; no longer C10.-, C11.-, C9.-
- net IR_OUT1: now also U1.37
- net IR_OUT2: now also U1.38
- net IR_OUT3: now also U1.39; no longer U1.37
- net IR_OUT4: now also U1.40; no longer U1.38
- net LED1: now also U1.24; no longer U1.39
- net LED2: now also U1.25; no longer U1.40
- net LED3: now also U1.26
- net LED4: now also U1.27
- net STBY: now also U5.19
- net VCC: now also C11.1; no longer C11.+, U5.19
- net VDD: now also C10.1; no longer C10.+
Routing:
- net VCC: track 132.9 -> 128.5 mm
- net 5V: track 28.1 -> 26.8 mm
- net VDD: track 31.0 -> 30.4 mm

Commit message: meet update 2
Parts:
- R11, R12, R13, R14, R15, R16, R17, R18, R19, R20, R21, R22, R3, R4, R5, R6, R7, R8, R9: device resistor:R0603 -> SparkFun-Resistors:0805
Connections:
- net VCC: now also U1.1

Commit message: meet update 3
Parts:
- moved S2 117.1 mm to (94.2, 20.3)
- moved S1 117.0 mm to (108.2, 13.2)
- moved R22 108.1 mm to (101.9, 11.2)
- moved R21 104.4 mm to (98.8, 12.7)
- moved R20 104.3 mm to (99.8, 14.7)
- moved LED6 103.0 mm to (109.2, 52.3)
- moved R19 101.0 mm to (98.3, 14.7)
- moved LED7 97.4 mm to (110.0, 39.1)
- moved R15 97.4 mm to (109.7, 31.8)
- moved R17 97.4 mm to (109.7, 24.6)
- moved R18 97.4 mm to (109.7, 21.1)
- moved LED8 97.4 mm to (110.0, 35.3)
- moved R16 97.4 mm to (109.7, 28.2)
- moved R14 94.8 mm to (104.9, 52.3)
- moved R12 91.8 mm to (104.6, 55.1)
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Routing:
- net VCC: track 128.5 -> 8.17 mm, vias 7 -> 0
- net GND: track 94.5 -> 15.2 mm, vias 13 -> 0
- net V_BATT: track 45.4 -> 0.00 mm
- net M1CA: track 38.8 -> 0.00 mm, vias 1 -> 0
- net M1CB: track 37.0 -> 0.00 mm, vias 1 -> 0
- net VDD: track 30.4 -> 0.00 mm, vias 2 -> 0
- net RST: track 27.6 -> 0.00 mm, vias 1 -> 0
- net 5V: track 26.8 -> 0.00 mm, vias 2 -> 0
- net M1+: track 20.9 -> 0.00 mm
- net M2CB: track 18.1 -> 0.00 mm
- net M1-: track 16.0 -> 0.00 mm
- net JTAG-TMS: track 15.4 -> 0.00 mm, vias 2 -> 0
- net M2CA: track 14.4 -> 0.00 mm
- net USART1_TX: track 12.5 -> 0.00 mm, vias 2 -> 0
- net M2+: track 12.4 -> 0.00 mm
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Other:
- board size 48.8 x 69.3 mm -> 71.1 x 45.7 mm

Commit message: meet update 4
Parts:
- moved S2 40.4 mm to (134.4, 15.5)
- moved S1 32.2 mm to (137.9, 25.7)
- moved C19 18.2 mm to (81.5, 26.8), turned to 270 degrees
- moved Q3 13.9 mm to (81.8, 66.5), turned to 180 degrees
- moved C8 3.78 mm to (89.9, 10.2)
- moved IC1 2.90 mm to (83.6, 10.4)
- moved Q1 2.03 mm to (81.7, 44.7)
- moved U5 1.37 mm to (87.9, 27.4)
- moved C13 1.05 mm to (88.4, 34.4)
- moved R4 0.57 mm to (75.9, 61.0)
- moved C12 0.51 mm to (81.5, 49.0)

Commit message: meet update 5
Parts:
- C14: value 10uF, 33m<ESR<2.2 -> 10uF
- moved C4 30.0 mm to (96.0, 32.6), turned to 0 degrees
- moved R6 25.5 mm to (105.7, 55.9), turned to 0 degrees
- moved R12 23.1 mm to (84.3, 66.0), turned to 270 degrees
- moved U5 21.5 mm to (71.1, 40.9), turned to 270 degrees
- moved C5 18.2 mm to (82.5, 49.0)
- moved R9 15.9 mm to (88.4, 71.9), turned to 0 degrees
- moved R13 15.5 mm to (94.2, 66.0), turned to 270 degrees
- moved C1 9.52 mm to (99.6, 38.4)
- moved C3 9.16 mm to (82.3, 35.1)
- moved C13 8.74 mm to (81.3, 39.5)
- moved C17 8.59 mm to (80.3, 22.6)
- moved R8 8.53 mm to (84.3, 71.9), turned to 180 degrees
- moved C2 8.30 mm to (101.6, 38.4)
- moved Q5 8.12 mm to (106.7, 53.3), turned to 90 degrees
- moved U3 7.42 mm to (70.1, 48.3)
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Connections:
- net M2I1: now also U1.21; no longer U1.20
- net M2I2: now also U1.22; no longer U1.21
- net M2P: now also U1.23; no longer U1.22
- net STBY: now also U1.20; no longer U1.23
Routing:
- net 5V: track 0.00 -> 90.7 mm
- net M2P: track 0.00 -> 19.6 mm, vias 0 -> 2
- net M2I1: track 0.00 -> 19.1 mm, vias 0 -> 2
- net M2I2: track 0.00 -> 17.9 mm, vias 0 -> 2
- net STBY: track 0.00 -> 17.8 mm, vias 0 -> 2
- net M1I1: track 0.00 -> 15.1 mm, vias 0 -> 2
- net M1P: track 0.00 -> 12.8 mm, vias 0 -> 2
- net M1I2: track 0.00 -> 12.8 mm, vias 0 -> 2
- net VCC: track 8.17 -> 17.5 mm
- net IR_IN3: track 0.00 -> 9.03 mm
- net IR_IN2: track 0.00 -> 9.03 mm
- net N$7: track 0.00 -> 8.43 mm
- net N$2: track 0.00 -> 6.81 mm
- net N$4: track 0.00 -> 6.73 mm
- net N$5: track 0.00 -> 6.73 mm
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
Commit message: meet update 6
Parts:
- added C22: 10uF, SparkFun-Capacitors:0805
- C9: value 20uF -> 10uF
- moved S2 40.4 mm to (95.2, 25.7)
- moved C2 20.6 mm to (81.0, 38.4), turned to 180 degrees
- moved R18 20.5 mm to (101.6, 39.9), turned to 180 degrees
- moved C6 19.6 mm to (83.3, 49.7), turned to 90 degrees
- moved C1 18.6 mm to (81.0, 39.9), turned to 180 degrees
- moved C5 17.7 mm to (100.1, 46.5), turned to 270 degrees
- moved C10 16.8 mm to (84.2, 35.6), turned to 270 degrees
- moved U2 16.7 mm to (81.0, 35.3)
- moved C3 14.9 mm to (85.3, 49.7), turned to 90 degrees
- moved LED5 14.3 mm to (104.9, 34.5), turned to 180 degrees
- moved R17 14.2 mm to (101.6, 36.3), turned to 180 degrees
- moved C7 14.2 mm to (88.4, 34.5)
- moved R16 12.8 mm to (101.6, 38.1), turned to 180 degrees
- moved LED6 11.1 mm to (104.9, 36.3), turned to 180 degrees
- moved R15 8.59 mm to (101.6, 34.5), turned to 180 degrees
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Connections:
- net 5V: now also C22.1
- net GND: now also C22.2
Routing:
- net GND: track 17.4 -> 26.8 mm
- net VCC: track 17.5 -> 24.3 mm
- net VDD: track 0.00 -> 5.75 mm
- net N$6: track 2.32 -> 7.60 mm
- net I2C1_SCL: track 15.0 -> 16.8 mm
- net I2C1_SDA: track 15.3 -> 17.1 mm
- net N$2: track 6.81 -> 5.07 mm
- net INT: track 6.44 -> 8.11 mm

Commit message: meet update 7
Parts:
- added X1: 22-23-2031, battery_plug:22-23-2031
- R11, R12, R13, R14: value (none) -> 2k
- R3, R4, R5, R6: value (none) -> 160 Ohm
- moved S1 42.8 mm to (98.0, 10.2), turned to 180 degrees
- moved C17 25.4 mm to (70.9, 46.2), turned to 180 degrees
- moved S2 18.7 mm to (105.7, 10.2), turned to 180 degrees
- moved C14 14.2 mm to (92.5, 9.91)
- moved C8 10.7 mm to (79.2, 9.91), turned to 90 degrees
- moved C15 9.33 mm to (69.6, 34.7), turned to 0 degrees
- moved R20 8.13 mm to (108.0, 14.7)
- moved C19 7.85 mm to (75.9, 34.0), turned to 0 degrees
- moved C9 6.61 mm to (73.9, 48.5)
- moved R21 5.95 mm to (104.4, 14.7), turned to 180 degrees
- moved JP4 5.02 mm to (99.1, 19.1)
- moved R22 3.70 mm to (100.8, 14.7)
- moved C11 2.75 mm to (67.7, 48.5), turned to 90 degrees
- moved C22 2.27 mm to (75.9, 35.8), turned to 180 degrees
- moved IC1 2.09 mm to (85.6, 9.91), turned to 270 degrees
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Connections:
- net 5V: now also R3.2, R4.2, R5.2, R6.2; no longer LED1.A, LED2.A, LED3.A, LED4.A
- net GND: now also LED1.K, LED2.K, LED3.K, LED4.K, X1.3; no longer R3.1, R4.1, R5.1, R6.1
- net M1+: now also JP4.1; no longer JP3.2
- net M1-: now also JP4.2; no longer JP3.1
- net M2+: now also JP3.1; no longer JP4.2
- net M2-: now also JP3.2; no longer JP4.1
- net N$14: now also LED4.A, Q5.3; no longer Q2.3, R3.2
- net N$15: now also Q2.2, R3.1; no longer Q3.3, R4.2
- net N$16: now also Q4.2, R5.1; no longer Q4.3, R5.2
- net N$17: now also Q5.2, R6.1; no longer Q5.3, R6.2
- net N$3: now also Q3.2, R4.1; no longer LED1.K, Q2.2
- net N$4: now also LED1.A, Q2.3; no longer LED2.K, Q3.2
- net N$5: now also LED2.A, Q3.3; no longer LED3.K, Q4.2
- net N$7: now also LED3.A, Q4.3; no longer LED4.K, Q5.2
- net V_BATT: now also X1.1
Routing:
- net V_BATT: track 0.00 -> 68.7 mm
- net VCC: track 24.3 -> 33.5 mm, vias 0 -> 2
- net GND: track 26.8 -> 35.6 mm
- net N$7: track 8.43 -> 0.00 mm
- net N$3: track 8.43 -> 0.00 mm
- net N$4: track 6.73 -> 0.00 mm
- net N$5: track 6.73 -> 0.00 mm
- net 5V: track 90.7 -> 97.4 mm
- net VDD: track 5.75 -> 10.5 mm
- net N$16: track 2.99 -> 0.00 mm
- net N$15: track 2.89 -> 0.00 mm
- net N$17: track 2.53 -> 0.00 mm
- net N$14: track 1.88 -> 0.00 mm

Commit message: sleep save
Parts:
- removed LED8: (no value), eagle-ltspice:LED_SML0603
- removed R18, R20, R21: (no value), SparkFun-Resistors:0805
- removed S2: DTS-3, switch-tact copy:DTS-3
- removed SWD: (no value), SparkFun-Connectors:1X05_LOCK
- removed USART: (no value), SparkFun-Connectors:1X04_LOCK
- added U$1: M04X2, SparkFun-Connectors:2X4
- moved C19 9.66 mm to (66.3, 34.3), turned to 90 degrees
- moved R19 7.47 mm to (104.4, 12.4), turned to 0 degrees
- moved R14 6.97 mm to (104.6, 54.9), turned to 180 degrees
- moved R3 6.51 mm to (68.3, 53.3), turned to 0 degrees
- moved R22 5.99 mm to (104.4, 9.91)
- moved R11 4.13 mm to (68.3, 51.8)
- moved C12 3.61 mm to (79.7, 46.4), turned to 90 degrees
- moved R6 2.74 mm to (104.6, 53.3), turned to 180 degrees
- moved Q2 2.54 mm to (63.5, 53.3), turned to 90 degrees
- moved Q5 2.54 mm to (109.2, 53.3), turned to 270 degrees
- moved LED7 1.78 mm to (104.9, 38.1)
- moved R16 1.78 mm to (101.6, 36.3)
- moved R17 1.78 mm to (101.6, 38.1)
- moved C22 0.80 mm to (76.2, 35.1), turned to 270 degrees
- moved C15 0.76 mm to (70.4, 34.7), turned to 180 degrees
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Connections:
- removed net BUTTON2: R20.2, U1.30
- removed net N$29: LED8.A, R16.1
- removed net N$30: R20.1, R21.1, S2.1
- net GND: now also U$1.8; no longer LED8.C, R21.2, SWD.1, USART.1
- net JTAG-TCK: now also U$1.5; no longer SWD.3
- net JTAG-TDO: now also U$1.7; no longer SWD.2
- net JTAG-TMS: now also U$1.3; no longer SWD.4
- net LED2: now also R16.2; no longer R17.2
- net LED3: now also R17.2; no longer R18.2
- net LED4: no longer R16.2
- net N$27: now also R16.1; no longer R17.1
- net N$28: now also R17.1; no longer R18.1
- net RST: now also U$1.1; no longer SWD.5
- net USART1_RX: now also U$1.4; no longer USART.3
- net USART1_TX: now also U$1.6; no longer USART.2
- net VCC: now also U$1.2; no longer S2.2, USART.4
Routing:
- net GND: track 35.6 -> 183.0 mm, vias 0 -> 9
- net VCC: track 33.5 -> 169.4 mm, vias 2 -> 5
- net M1+: track 0.00 -> 48.6 mm, vias 0 -> 1
- net M1-: track 0.00 -> 47.7 mm, vias 0 -> 1
- net V_BATT: track 68.7 -> 23.4 mm
- net M2-: track 0.00 -> 43.4 mm, vias 0 -> 1
- net M2+: track 0.00 -> 42.0 mm, vias 0 -> 1
- net 5V: track 97.4 -> 61.6 mm, vias 0 -> 1
- net M2CB: track 0.00 -> 32.7 mm
- net M2CA: track 0.00 -> 26.0 mm
- net IR_OUT3: track 0.00 -> 23.5 mm, vias 0 -> 2
- net USART1_TX: track 0.00 -> 15.5 mm, vias 0 -> 1
- net RST: track 0.00 -> 14.8 mm
- net LED1: track 0.00 -> 14.7 mm
- net LED2: track 0.00 -> 14.6 mm
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- added copper zone on layer 1, net GND
